File: HARDWARE/ESP32-C5-DevKit-Lipo-Rev.A/ESP32-C5-DevKit-Lipo_Rev_A.kicad_pcb (KiCad board)
At the start: 2 copper layers, 25.4 x 53.6 mm, 86 parts, among them T1 BC817-40(SOT23), T2 BC817-40(SOT23), U1 TP4054-42-SOT25-R, U2 CH340X(MSOP-10), U3 ESP32-C5-WROOM-1-N8R4

Commit message: Update
Improved battery measurement circuit before board release
Parts:
- R21: value 1k/R0402 -> 0R/R0402
Changed lines of the file:
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@@
         (effects (font (size 0.762 0.762) (thickness 0.1905)) (justify mirror))
     )
-    (fp_text value "1k/R0402" (at 0 -1.5) (layer "B.Fab")
+    (fp_text value "0R/R0402" (at 0 -1.5) (layer "B.Fab")
         (effects (font (size 1.27 1.27) (thickness 0.254)) (justify mirror))
     )
